Commit message: 测试物体换圆柱、删一键抓取脚本、夹取检测改用夹爪角度、Gazebo 材质上色
- cube.urdf -> cylinder.urdf(r=1.5cm h=6cm 竖立),launch/脚本/README 同步
- 删除 grasp_cube.py:固定 spawn 坐标会被腕关节漂移带偏,维护价值低,
  手动夹取用 manual_control.py 足够
- manual_control: 夹取检测从读 /model_states+/link_states 位姿改为
  看夹爪关节角度(空夹合到下限 -0.1745,夹到东西停得更开),
  去掉 link_states 订阅;夹爪开合 effort 符号修正(负值闭合)
- Gazebo Classic 忽略 URDF <material><color>,按 link 加
  Gazebo/Yellow(臂)/Gazebo/Black(夹爪)材质标签
- 问题排查记录精简为 现象/原因/解决办法 三段式,PID 条目
  注明详见 so101_moveit_mujoco 的 control_basics.md

File: src/so101_moveit_gazebo/urdf/so101_gazebo.urdf.xacro (robot description, xacro)
@@ -11,4 +11,14 @@
   <!-- 机器人本体（公共描述） -->
   <xacro:so101_description/>
+  <!-- Gazebo Classic 材质：它忽略 URDF 的 <material><color>，只对整 link 应用
+       自己的命名材质。黄 = 打印结构件，黑 = 舵机/夹爪，与 RViz 里 3d_printed/sts3215 对应。 -->
+  <gazebo reference="base_link"><material>Gazebo/Yellow</material></gazebo>
+  <gazebo reference="shoulder_link"><material>Gazebo/Yellow</material></gazebo>
+  <gazebo reference="upper_arm_link"><material>Gazebo/Yellow</material></gazebo>
+  <gazebo reference="lower_arm_link"><material>Gazebo/Yellow</material></gazebo>
+  <gazebo reference="wrist_link"><material>Gazebo/Yellow</material></gazebo>
+  <gazebo reference="gripper_link"><material>Gazebo/Black</material></gazebo>
+  <gazebo reference="gripper_frame_link"><material>Gazebo/Black</material></gazebo>
+  <gazebo reference="moving_jaw_so101_v1_link"><material>Gazebo/Black</material></gazebo>
   <!-- Gazebo 专用：world 虚链接 + fixed 关节，把整机焊死在空中，
        防止底盘倾倒/滑动，同时消除 KDL 根链接带惯性的警告。 -->
