Commit message: 接入 MoveIt Servo 实时微动：moveit_config(srdf/运动学/限位/servo参数)、servo launch、URDF关节damping、接入记录文档
- moveit_config/: so101.srdf、kinematics/joint_limits/moveit_controllers/pilz配置、servo_parameters.yaml(2.5.9平铺格式,5DOF奇异阈值实测标定)
- so101_moveit_servo.launch.py: Servo节点+PlanningScene,输出接Gazebo JTC(100Hz对齐)
- so101_description.xacro: 5臂关节加damping=1.0,压Servo静止时重力下坠抖动
- doc/moveit_servo_接入记录.md: 参数格式、JointJog stamp、双通道互斥、/clock量化告警等踩坑
- README/文件说明: 已完成Servo接入与直接操控(joint_teleop/ee_teleop手柄遥操),TODO改为MoveIt规划器

File: src/so101_moveit_gazebo/urdf/so101_description.xacro (robot description, xacro)
@@ -332,4 +332,6 @@
       <axis xyz="0 0 1"/>
       <limit effort="10" velocity="10" lower="-2.74385" upper="2.84121"/>
+      <!-- 粘性阻尼：压传送窗口内的重力下坠速度，消除 Servo 静止时的可见抖动 -->
+      <dynamics damping="1.0"/>
     </joint>
     <!-- Joint from lower_arm to wrist -->
@@ -340,4 +342,5 @@
       <axis xyz="0 0 1"/>
       <limit effort="10" velocity="10" lower="-1.65806" upper="1.65806"/>
+      <dynamics damping="1.0"/>
     </joint>
     <!-- Joint from upper_arm to lower_arm -->
@@ -349,4 +352,5 @@
       <axis xyz="0 0 1"/>
       <limit effort="10" velocity="10" lower="-1.69" upper="1.69"/>
+      <dynamics damping="1.0"/>
     </joint>
     <!-- Joint from shoulder to upper_arm -->
@@ -357,4 +361,5 @@
       <axis xyz="0 0 1"/>
       <limit effort="10" velocity="10" lower="-1.74533" upper="1.74533"/>
+      <dynamics damping="1.0"/>
     </joint>
     <!-- Joint from base to shoulder -->
@@ -365,4 +370,5 @@
       <axis xyz="0 0 1"/>
       <limit effort="10" velocity="10" lower="-1.91986" upper="1.91986"/>
+      <dynamics damping="1.0"/>
     </joint>
   </xacro:macro>
